Commit message: changes to circle size

File: husky/husky_description/urdf/husky_macro.urdf.xacro (robot description, xacro)
@@ -90,5 +90,5 @@
     <link name="${prefix}imu_link"/>
     <joint name="${prefix}imu_joint" type="fixed">
-      <origin xyz="$(optenv CPR_IMU_XYZ 0 0 0)" rpy="$(optenv CPR_IMU_RPY 0 0 0)" />
+      <origin xyz="" rpy="$(optenv CPR_IMU_RPY 0 0 0)" />
       <parent link="${prefix}base_link" />
       <child link="${prefix}imu_link" />
